File: multivibrator.sch (KiCad schematic (older format))
At the start: 11 parts, among them CON1 BARREL_JACK, Q1 Q_NPN_BCE, Q2 Q_NPN_BCE

Commit message: switch transsitor footprint
Parts:
- Q1, Q2: value Q_NPN_BCE -> Q_NPN_EBC; footprint Transistors_OldSowjetAera:OldSowjetaera_Transistor_Type-I_BigPads -> TO_SOT_Packages_THT:TO-92_Inline_Narrow_Oval; symbol Q_NPN_BCE -> Q_NPN_EBC
Connections:
- net at C1.1, R1.2: now also Q1.3 (C); no longer Q1.2 (C)
- net at C1.2, R2.2: now also Q2.2 (B); no longer Q2.1 (B)
- net at C2.2, R3.2: now also Q1.2 (B); no longer Q1.1 (B)
- net at C2.1, R4.2: now also Q2.3 (C); no longer Q2.2 (C)
- net at D1.2 (A): now also Q1.1 (E); no longer Q1.3 (E)
- net at D2.2 (A): now also Q2.1 (E); no longer Q2.3 (E)
Changed lines of the file:
@@
 $EndComp
 $Comp
-L Q_NPN_BCE Q1
+L Q_NPN_EBC Q1
 U 1 1 57D00F4C
 P 2750 3050
 F 0 "Q1" H 3050 3100 50  0000 R CNN
-F 1 "Q_NPN_BCE" H 3350 3000 50  0000 R CNN
-F 2 "Transistors_OldSowjetAera:OldSowjetaera_Transistor_Type-I_BigPads" H 2950 3150 50  0001 C CNN
+F 1 "Q_NPN_EBC" H 3350 3000 50  0000 R CNN
+F 2 "TO_SOT_Packages_THT:TO-92_Inline_Narrow_Oval" H 2950 3150 50  0001 C CNN
 F 3 "" H 2750 3050 50  0000 C CNN
 	1    2750 3050
@@
 $EndComp
 $Comp
-L Q_NPN_BCE Q2
+L Q_NPN_EBC Q2
 U 1 1 57D00F94
 P 3950 3050
 F 0 "Q2" H 4250 3100 50  0000 R CNN
-F 1 "Q_NPN_BCE" H 4550 3000 50  0000 R CNN
-F 2 "Transistors_OldSowjetAera:OldSowjetaera_Transistor_Type-I_BigPads" H 4150 3150 50  0001 C CNN
+F 1 "Q_NPN_EBC" H 4550 3000 50  0000 R CNN
+F 2 "TO_SOT_Packages_THT:TO-92_Inline_Narrow_Oval" H 4150 3150 50  0001 C CNN
 F 3 "" H 3950 3050 50  0000 C CNN
 	1    3950 3050

Commit message: ebc npn transistors laid out
Parts:
- Q1, Q2: footprint TO_SOT_Packages_THT:TO-92_Inline_Narrow_Oval -> TO_SOT_Packages_THT:TO-92_Inline_Wide
Changed lines of the file:
@@
 F 0 "Q1" H 3050 3100 50  0000 R CNN
 F 1 "Q_NPN_EBC" H 3350 3000 50  0000 R CNN
-F 2 "TO_SOT_Packages_THT:TO-92_Inline_Narrow_Oval" H 2950 3150 50  0001 C CNN
+F 2 "TO_SOT_Packages_THT:TO-92_Inline_Wide" H 2950 3150 50  0001 C CNN
 F 3 "" H 2750 3050 50  0000 C CNN
 	1    2750 3050
@@
 F 0 "Q2" H 4250 3100 50  0000 R CNN
 F 1 "Q_NPN_EBC" H 4550 3000 50  0000 R CNN
-F 2 "TO_SOT_Packages_THT:TO-92_Inline_Narrow_Oval" H 4150 3150 50  0001 C CNN
+F 2 "TO_SOT_Packages_THT:TO-92_Inline_Wide" H 4150 3150 50  0001 C CNN
 F 3 "" H 3950 3050 50  0000 C CNN
 	1    3950 3050
